Commit message: Intel R200 point cloud plotting

File: ros_camera_sweep/urdf/sweep.urdf (robot description, URDF)
Before this commit: robot camera_sweep, 2 links, 1 joints
Joints:
- joint camera_base_to_camera_link_joint: origin xyz=0 0 0 -> xyz=-0.0364 0 0.0296

Commit message: Updated package path in launch files.

File: ros_camera_sweep/urdf/sweep.urdf (robot description, URDF)
Before this commit: robot camera_sweep, 2 links, 1 joints
Links:
- removed link camera_link
- added link camera_mount; visual mesh filename=package://ros_camera_sweep/meshes/camera.stl
Joints:
- joint camera_base_to_camera_link_joint: child camera_link -> camera_mount; type fixed -> floating
